Commit message: editing urdf model and importing models folder

File: bumperbot_ws/src/bumperbot_description/urdf/bumperbot.urdf.xacro (robot description, xacro)
@@ -1,71 +1,146 @@
 <?xml version="1.0"?>
-<robot xmlns:xacro="http://www.ros.org/wiki/xacro" name="bumperbot">
-    <link name="base_footprint"/>
-    <link name="base_link">
-        <visual>
-            <origin rpy="0 0 0" xyz="0 0 0"/> <!-- indicate the orientation and the position of the mesh base_link.STL with respect to the base_link -->
-            <geometry>
-                <mesh filename="package://bumperbot_description/meshes/base_link.STL"/>
-            </geometry>
-        </visual>
-    </link>
-    <joint name="base_joint" type="fixed">
-        <parent link="base_footprint"/>
-        <child link="base_link"/>
-        <origin rpy="0 0 0" xyz="0 0 0.033"/> <!-- indicate the orientation and the position between two reference frames between two links -->
-    </joint>
-    <link name="wheel_right_link">
-        <visual>
-            <origin rpy="1.57 0 0" xyz="0 0 0"/>
-            <geometry>
-                <mesh filename="package://bumperbot_description/meshes/wheel_right_link.STL"/>
-            </geometry>
-        </visual>
-    </link>
-    <joint name="wheel_right_joint" type="continuous">
-        <parent link="base_link"/>
-        <child link="wheel_right_link"/>
-        <axis xyz="0 1 0"/>
-        <origin rpy="0 0 0" xyz="0 -0.07 0"/>
-    </joint>
-    <link name="wheel_left_link">
-        <visual>
-            <origin rpy="-1.57 0 0" xyz="0 0 0"/>
-            <geometry>
-                <mesh filename="package://bumperbot_description/meshes/wheel_left_link.STL"/>
-            </geometry>
-        </visual>
-    </link>
-    <joint name="wheel_left_joint" type="continuous">
-        <parent link="base_link"/>
-        <child link="wheel_left_link"/>
-        <axis xyz="0 1 0"/>
-        <origin rpy="0 0 0" xyz="0 0.07 0"/>
-    </joint>
-    <link name="caster_front_link">
-        <visual>
-            <origin rpy="0 0 0" xyz="0 0 0"/>
-            <geometry>
-                <mesh filename="package://bumperbot_description/meshes/caster_front_link.STL"/>
-            </geometry>
-        </visual>
-    </link>
-    <joint name="caster_front_joint" type="fixed">
-        <parent link="base_link"/>
-        <child link="caster_front_link"/>
-        <origin rpy="0 0 0" xyz="0.04755 0.0 -0.0275"/>
-    </joint>
-    <link name="caster_rear_link">
-        <visual>
-            <origin rpy="0 0 0" xyz="0 0 0"/>
-            <geometry>
-                <mesh filename="package://bumperbot_description/meshes/caster_rear_link.STL"/>
-            </geometry>
-        </visual>
-    </link>
-    <joint name="caster_rear_joint" type="fixed">
-        <parent link="base_link"/>
-        <child link="caster_rear_link"/>
-        <origin rpy="0 0 0" xyz="-0.04755 0.0 -0.0275"/>
-    </joint>
+<robot name="bumperbot" xmlns:xacro="http://ros.org/wiki/xacro">
+  <!-- Include Gazebo Parameters -->
+  <xacro:include filename="$(find bumperbot_description)/urdf/bumperbot_gazebo.xacro" />
+  <link name="base_footprint"/>
+  <link name="base_link">
+    <!-- inertial tag is required for the gazebo simulation-->
+    <inertial>
+      <origin xyz="0 0 0.04" rpy="0.0 0.25 0.3" />
+      <mass value="8.2573504e-01"/>
+      <inertia ixx="2.2124416e-02" ixy="-1.2294101e-04" ixz="3.4938785e-04"
+               iyy="2.1193702e-02" iyz="-5.0120904e-05"
+               izz="2.0064271e-02" />
+    </inertial>
+    <visual>
+      <origin xyz="0 0 0" rpy="0 0 0" /> <!-- indicate the orientation and the position of the mesh base_link.STL with respect to the base_link -->
+      <geometry>
+        <mesh filename="package://bumperbot_description/meshes/base_link.STL" />
+      </geometry>
+    </visual>
+    <!-- collision tag is required for the gazebo simulation-->
+    <collision>
+      <origin xyz="0 0 0" rpy="0 0 0" /> <!-- indicate the orientation and the position of the mesh base_link.STL with respect to the base_link -->
+      <geometry>
+        <!-- we will use another thing to describe the geometry of the wheel beacuse stl is very expensive to simulate while the wheel is rotating -->
+        <!-- <mesh filename="package://bumperbot_description/meshes/wheel_right_link.STL"/> -->
+        <mesh filename="package://bumperbot_description/meshes/base_link.STL" />
+      </geometry>
+    </collision>
+  </link>
+  <joint name="base_joint" type="fixed">
+    <parent link="base_footprint"/>
+    <child link="base_link" />
+    <origin xyz="0 0 0.033" rpy="0 0 0"/> <!-- indicate the orientation and the position between two reference frames between two links -->
+  </joint>
+  <link name="wheel_right_link">
+    <!-- inertial tag is required for the gazebo simulation-->
+    <inertial>
+      <origin xyz="0 -0.014 0" rpy="0 0 0" />
+      <mass value="0.0530086090966721" />
+      <inertia ixx="1.88176298336665E-05" ixy="-4.8444933029987E-10" ixz="1.88163708851143E-08"
+               iyy="3.11510738647764E-05" iyz="-6.93560663069607E-11"
+               izz="1.8801969558182E-05" />
+    </inertial>
+    <visual>
+      <origin xyz="0 0 0" rpy="1.57 0 0" />
+      <geometry>
+        <mesh filename="package://bumperbot_description/meshes/wheel_right_link.STL" />
+      </geometry>
+    </visual>
+    <collision>
+      <origin xyz="0 -0.015 0" rpy="1.57 0 0" />
+      <geometry>
+        <sphere radius="0.033"/>
+      </geometry>
+    </collision>
+  </link>
+  <joint name="wheel_right_joint" type="continuous">
+    <origin xyz="0 -0.0701101849418637 0" rpy="0 0 0" />
+    <parent link="base_link" />
+    <child link="wheel_right_link" />
+    <axis xyz="0 1 0" />
+  </joint>
+  <link
+    name="wheel_left_link">
+    <inertial>
+      <origin xyz="0 0.014 0" rpy="0 0 0" />
+      <mass value="0.0530086043217644" />
+      <inertia ixx="1.8792911368909E-05"  ixy="3.31256392204584E-10" ixz="-1.14082001662767E-08"
+               iyy="3.11510738759073E-05" iyz="-3.60499245082192E-10"
+               izz="1.88266886146847E-05" />
+    </inertial>
+    <visual>
+      <origin xyz="0 0 0" rpy="-1.57 0 0" />
+      <geometry>
+        <mesh filename="package://bumperbot_description/meshes/wheel_left_link.STL" />
+      </geometry>
+    </visual>
+    <collision>
+      <origin xyz="0 0.015 0" rpy="-1.57 0 0" />
+      <geometry>
+        <sphere radius="0.033"/>
+      </geometry>
+    </collision>
+  </link>
+  <joint name="wheel_left_joint" type="continuous">
+    <origin xyz="0 0.0701101849418642 0" rpy="0 0 0" />
+    <parent link="base_link" />
+    <child link="wheel_left_link" />
+    <axis xyz="0 1 0" />
+  </joint>
+  <link name="caster_front_link">
+    <inertial>
+      <origin xyz="3.89968128948481E-07 2.40073004698083E-07 0.00219173397061506" rpy="0 0 0" />
+      <mass value="1.44379265037903E-06" />
+      <inertia ixx="7.23075276010246E-11" ixy="-6.10956883467859E-16" ixz="2.22849693525031E-15"
+               iyy="3.8713793085917E-11"  iyz="2.93909858781952E-15"
+               izz="1.00967486676306E-10" />
+    </inertial>
+    <visual>
+      <origin xyz="0 0 0" rpy="0 0 0" />
+      <geometry>
+        <mesh filename="package://bumperbot_description/meshes/caster_front_link.STL" />
+      </geometry>
+    </visual>
+    <collision>
+      <origin xyz="0 0 0" rpy="0 0 0" />
+      <geometry>
+        <sphere radius="0.005"/>
+      </geometry>
+    </collision>
+  </link>
+  <joint name="caster_front_joint" type="fixed">
+    <origin xyz="0.04755 0 -0.0275" rpy="0 0 0" />
+    <parent link="base_link" />
+    <child link="caster_front_link" />
+    <axis xyz="0 0 0" />
+  </joint>
+  <link name="caster_rear_link">
+    <inertial>
+      <origin xyz="3.8996812895542E-07 2.40073004698083E-07 0.00219173397061509" rpy="0 0 0" />
+      <mass value="1.44379265037902E-06" />
+      <inertia ixx="7.23075276010246E-11" ixy="-6.10956872363424E-16" ixz="2.22849693527207E-15"
+               iyy="3.87137930859167E-11" iyz="2.939098587861E-15"
+               izz="1.00967486676306E-10" />
+    </inertial>
+    <visual>
+      <origin xyz="0 0 0" rpy="0 0 0" />
+      <geometry>
+        <mesh filename="package://bumperbot_description/meshes/caster_rear_link.STL" />
+      </geometry>
+    </visual>
+    <collision>
+      <origin xyz="0 0 0" rpy="0 0 0" />
+      <geometry>
+        <sphere radius="0.005"/>
+      </geometry>
+    </collision>
+  </link>
+  <joint name="caster_rear_joint" type="fixed">
+    <origin xyz="-0.04755 0 -0.0275" rpy="0 0 0" />
+    <parent link="base_link" />
+    <child link="caster_rear_link" />
+    <axis xyz="0 0 0" />
+  </joint>
 </robot>

Commit message: adding gazebo controller

File: bumperbot_ws/src/bumperbot_description/urdf/bumperbot.urdf.xacro (robot description, xacro)
@@ -3,4 +3,5 @@
   <!-- Include Gazebo Parameters -->
   <xacro:include filename="$(find bumperbot_description)/urdf/bumperbot_gazebo.xacro" />
+  <xacro:include filename="$(find bumperbot_description)/urdf/bumperbot_ros2_control.xacro" />
   <link name="base_footprint"/>
   <link name="base_link">

File: bumperbot_ws/src/bumperbot_description/urdf/bumperbot_gazebo.xacro (robot description, xacro)
@@ -1,4 +1,20 @@
 <?xml version="1.0"?>
 <robot name="bumperbot" xmlns="http://ros.org/wiki/xacro">
+    <!-- this tag indicates the presence of a mechanical transmission that connects each motor of the robot to each link of the wheel -->
+    <transmission>
+        <plugin>transmission_interface/SimpleTransmission</plugin>
+        <actuator name="wheel_right_motor" role="actuator_right"/>
+        <joint name="wheel_right_joint" role="joint_right">
+            <mechanical_reduction>1.0</mechanical_reduction> <!-- one degree of rotation of the motor corresponds to one degree of rotation of the wheel -->
+        </joint>
+    </transmission>
+    <!-- this tag indicates the presence of a mechanical transmission that connects each motor of the robot to each link of the wheel -->
+    <transmission>
+        <plugin>transmission_interface/SimpleTransmission</plugin>
+        <actuator name="wheel_left_motor" role="actuator_left"/>
+        <joint name="wheel_left_joint" role="joint_left">
+            <mechanical_reduction>1.0</mechanical_reduction> <!-- one degree of rotation of the motor corresponds to one degree of rotation of the wheel -->
+        </joint>
+    </transmission>
     <gazebo reference="wheel_right_link">
         <mu1>100000000000000.0</mu1>
@@ -35,3 +51,10 @@
         <maxVel>0.1</maxVel>
     </gazebo>
+    <gazebo>
+        <plugin filename="libgazebo_ros2_control.so" name="gazebo_ros2_control">
+            <robot_param>robot_description</robot_param>
+            <robot_param_node>robot_state_publisher</robot_param_node>
+            <parameters></parameters>
+        </plugin>
+    </gazebo>
 </robot>

Commit message: implementing controller and creating launch file

File: bumperbot_ws/src/bumperbot_description/urdf/bumperbot.urdf.xacro (robot description, xacro)
@@ -1,4 +1,4 @@
 <?xml version="1.0"?>
-<robot name="bumperbot" xmlns:xacro="http://ros.org/wiki/xacro">
+<robot name="bumperbot" xmlns:xacro="http://www.ros.org/wiki/xacro">
   <!-- Include Gazebo Parameters -->
   <xacro:include filename="$(find bumperbot_description)/urdf/bumperbot_gazebo.xacro" />

File: bumperbot_ws/src/bumperbot_description/urdf/bumperbot_gazebo.xacro (robot description, xacro)
@@ -1,6 +1,6 @@
 <?xml version="1.0"?>
-<robot name="bumperbot" xmlns="http://ros.org/wiki/xacro">
+<robot name="bumperbot" xmlns="http://www.ros.org/wiki/xacro">
     <!-- this tag indicates the presence of a mechanical transmission that connects each motor of the robot to each link of the wheel -->
-    <transmission>
+    <transmission name="wheel_right_transmission">
         <plugin>transmission_interface/SimpleTransmission</plugin>
         <actuator name="wheel_right_motor" role="actuator_right"/>
@@ -10,5 +10,5 @@
     </transmission>
     <!-- this tag indicates the presence of a mechanical transmission that connects each motor of the robot to each link of the wheel -->
-    <transmission>
+    <transmission name="wheel_left_transmission">
         <plugin>transmission_interface/SimpleTransmission</plugin>
         <actuator name="wheel_left_motor" role="actuator_left"/>
@@ -55,5 +55,5 @@
             <robot_param>robot_description</robot_param>
             <robot_param_node>robot_state_publisher</robot_param_node>
-            <parameters></parameters>
+            <parameters>$(find bumperbot_controller)/config/bumperbot_controllers.yaml</parameters>
         </plugin>
     </gazebo>

File: bumperbot_ws/src/bumperbot_description/urdf/bumperbot_ros2_control.xacro (robot description, xacro)
@@ -1,4 +1,4 @@
 <?xml version="1.0"?>
-<robot name="bumperbot" xmlns:xacro="http://ros.org/wiki/xacro">
+<robot name="bumperbot" xmlns:xacro="http://www.ros.org/wiki/xacro">
     <ros2_control type="system" name="RobotSystem">
         <hardware>
@@ -13,5 +13,5 @@
             <state_interface name="velocity"/>
         </joint>
-        <joint name="wheel_lrft_joint">
+        <joint name="wheel_left_joint">
             <command_interface name="velocity">
                 <param name="min">-1</param>

Commit message: implmeneting kalman filter

File: bumperbot_ws/src/bumperbot_description/urdf/bumperbot.urdf.xacro (robot description, xacro)
@@ -145,3 +145,29 @@
     <axis xyz="0 0 0" />
   </joint>
+  <link name="imu_link">
+    <inertial>
+      <origin xyz="-0.00552433659106688 0.000168210391520346 0.000514000497342681" rpy="0 0 0" />
+      <mass value="0.000528415362211671" />
+      <inertia ixx="1.46176048428261E-08" ixy="1.40015117949421E-10" ixz="-1.99633872937403E-12"
+               iyy="8.59662482954888E-09" iyz="7.52375112767959E-12"
+               izz="2.30279421279312E-08" />
+    </inertial>
+    <visual>
+      <origin xyz="0 0 0" rpy="0 0 0"/>
+      <geometry>
+        <mesh filename="package://bumperbot_description/meshes/imu_link.STL"/>
+      </geometry>
+    </visual>
+    <collision>
+      <origin xyz="0 0 0" rpy="0 0 0"/>
+      <geometry>
+        <mesh filename="package://bumperbot_description/meshes/imu_link.STL"/>
+      </geometry>
+    </collision>
+  </link>
+  <joint name="imu_joint" type="fixed">
+    <parent link="base_link"/>
+    <child link="imu_link"/>
+    <origin xyz="0 0 0.07" rpy="0 0 0"/>
+  </joint>
 </robot>

File: bumperbot_ws/src/bumperbot_description/urdf/bumperbot_gazebo.xacro (robot description, xacro)
@@ -58,3 +58,52 @@
         </plugin>
     </gazebo>
+    <gazebo reference="imu_link">
+        <sensor name="imu" type="imu">
+            <always_on>true</always_on>
+            <update_rate>100</update_rate>
+            <imu>
+                <angular_velocity>
+                    <x>
+                        <noise type="gaussian">
+                            <mean>0.0</mean>
+                            <stddev>2e-4</stddev>
+                        </noise>
+                    </x>
+                    <y>
+                        <noise type="gaussian">
+                            <mean>0.0</mean>
+                            <stddev>2e-4</stddev>
+                        </noise>
+                    </y>
+                    <z>
+                        <noise type="gaussian">
+                            <mean>0.0</mean>
+                            <stddev>2e-4</stddev>
+                        </noise>
+                    </z>
+                </angular_velocity>
+                <linear_acceleration>
+                    <x>
+                        <noise type="gaussian">
+                            <mean>0.0</mean>
+                            <stddev>1.7e-2</stddev>
+                        </noise>
+                    </x>
+                    <y>
+                        <noise type="gaussian">
+                            <mean>0.0</mean>
+                            <stddev>1.7e-2</stddev>
+                        </noise>
+                    </y>
+                    <z>
+                        <noise type="gaussian">
+                            <mean>0.0</mean>
+                            <stddev>1.7e-2</stddev>
+                        </noise>
+                    </z>
+                </linear_acceleration>
+            </imu>
+            <plugin name="imu" filename="libgazebo_ros_imu_sensor.so"/>
+        </sensor>
+    </gazebo>
 </robot>

Commit message: adding camera

File: bumperbot_ws/src/bumperbot_description/urdf/bumperbot.urdf.xacro (robot description, xacro)
@@ -171,3 +171,31 @@
     <origin xyz="0 0 0.07" rpy="0 0 0"/>
   </joint>
+  <link name="camera_link">
+    <inertial>
+      <mass value="0.1" />
+      <origin xyz="0 0 0" />
+      <inertia ixx="0.0001" ixy="0.0" ixz="0.0" iyy="0.0001" iyz="0.0" izz="0.0001" />
+    </inertial>
+    <visual>
+      <origin xyz="0.0 0.0 0.0" rpy="0 0 0"/>
+      <geometry>
+        <box size="0.05 0.05 0.1"/>
+      </geometry>
+      <material name="grey">
+        <color rgba="0.1 0.1 0.1 1.0"/>
+      </material>
+    </visual>
+    <collision>
+      <origin xyz="0 0 0.0" rpy="0 0 0"/>
+      <geometry>
+          <box size="0.05 0.05 0.1"/>
+      </geometry>
+    </collision>
+</link>
+<!-- Joint to attach camera to base_link (modify base_link to whatever link the camera is attached to) -->
+<joint name="camera_joint" type="fixed">
+    <parent link="base_link"/> <!-- Attach camera to the base or any other link -->
+    <child link="camera_link"/>
+    <origin xyz="0 0 0.15" rpy="0 0 0"/> <!-- Position relative to the robot -->
+</joint>
 </robot>

File: bumperbot_ws/src/bumperbot_description/urdf/bumperbot_gazebo.xacro (robot description, xacro)
@@ -107,3 +107,31 @@
         </sensor>
     </gazebo>
+    <gazebo reference="camera_link">
+        <sensor type="camera" name="camera_sensor">
+            <always_on>true</always_on>
+            <update_rate>30.0</update_rate>
+            <visualize>true</visualize>
+            <camera>
+                <horizontal_fov>1.047</horizontal_fov> <!-- Field of View (in radians) -->
+                <image>
+                    <width>640</width> <!-- Image width -->
+                    <height>480</height> <!-- Image height -->
+                    <format>R8G8B8</format> <!-- Image format -->
+                </image>
+                <clip>
+                    <near>0.1</near> <!-- Near clipping plane -->
+                    <far>100</far> <!-- Far clipping plane -->
+                </clip>
+            </camera>
+            <plugin name="camera_controller" filename="libgazebo_ros_camera.so">
+                <ros>
+                    <namespace>/camera</namespace>
+                    <argument>--ros-args</argument>
+                </ros>
+                <update_rate>30.0</update_rate>
+                <camera_name>bumperbot_camera</camera_name>
+                <frame_name>camera_link</frame_name>
+            </plugin>
+        </sensor>
+    </gazebo>
 </robot>
